File: kicad_source/R4CANAdapter.kicad_sch (KiCad schematic)
At the start: 35 parts, among them CN1 CONN_01X05, CN2 691322310004, CN3 GH_SM04B-GHS-TB, CN4 GH_SM04B-GHS-TB, CN5 SM04B-SRSS-TB, Q1 2N7002, Q2 2N7002, U1 MCP2551-I/SN, U2 24LC64

Commit message: updated images
Parts:
- U1, U2: footprint Package_SO:SO-8_3.9x4.9mm_P1.27mm -> Package_SO:SOIC-8_3.9x4.9mm_P1.27mm
Changed lines of the file:
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@@
       (effects (font (size 1.524 1.524)))
     )
-    (property "Footprint" "Package_SO:SO-8_3.9x4.9mm_P1.27mm" (id 2) (at 166.37 41.91 0)
+    (property "Footprint" "Package_SO:SOIC-8_3.9x4.9mm_P1.27mm" (id 2) (at 166.37 41.91 0)
       (effects (font (size 1.524 1.524)) hide)
     )
@@
       (effects (font (size 1.27 1.27)) (justify left))
     )
-    (property "Footprint" "Package_SO:SO-8_3.9x4.9mm_P1.27mm" (id 2) (at 181.61 134.62 0)
+    (property "Footprint" "Package_SO:SOIC-8_3.9x4.9mm_P1.27mm" (id 2) (at 181.61 134.62 0)
       (effects (font (size 1.27 1.27)) hide)
     )
@@
     )
     (path "/00000000-0000-0000-0000-00005fd751ff"
-      (reference "U1") (unit 1) (value "MCP2551-I/SN") (footprint "Package_SO:SO-8_3.9x4.9mm_P1.27mm")
+      (reference "U1") (unit 1) (value "MCP2551-I/SN") (footprint "Package_SO:SOIC-8_3.9x4.9mm_P1.27mm")
     )
     (path "/22be3d4d-ae12-4eb8-846f-0339b769d4f7"
-      (reference "U2") (unit 1) (value "24LC64") (footprint "Package_SO:SO-8_3.9x4.9mm_P1.27mm")
-    )
-  )
+      (reference "U2") (unit 1) (value "24LC64") (footprint "Package_SO:SOIC-8_3.9x4.9mm_P1.27mm")
+    )
+  )
